File: PDcharger/PDcharger.kicad_sch (KiCad schematic)
At the start: 0 parts

Commit message: ad
たしたよ。
Parts:
- added U1: TPS40057PWPR, TPS40057PWPR_footprints:PWP16_2P31X2P46-M, symbol 2026-06-10_10-14-18:TPS40057PWPR
Changed lines of the file:
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@@
 	(generator_version "10.0")
 	(paper "A4")
+	(symbol
+		(lib_id "2026-06-10_10-14-18:TPS40057PWPR")
+		(at 115.57 71.12 0)
+		(unit 1)
+		(body_style 1)
+		(exclude_from_sim no)
+		(in_bom yes)
+		(on_board yes)
+		(in_pos_files yes)
+		(dnp no)
+		(fields_autoplaced yes)
+		(property "Reference" "U1"
+			(at 148.59 60.96 0)
+			(show_name no)
+			(do_not_autoplace no)
+			(effects
+				(font
+					(size 1.524 1.524)
+				)
+			)
+		)
+		(property "Value" "TPS40057PWPR"
+			(at 148.59 63.5 0)
+			(show_name no)
+			(do_not_autoplace no)
+			(effects
+				(font
+					(size 1.524 1.524)
+				)
+			)
+		)
+		(property "Footprint" "TPS40057PWPR_footprints:PWP16_2P31X2P46-M"
+			(at 115.57 71.12 0)
+			(hide yes)
+			(show_name no)
+			(do_not_autoplace no)
+			(effects
+				(font
+					(size 1.27 1.27)
+					(italic yes)
+				)
+			)
+		)
+		(property "Datasheet" "https://www.ti.com/lit/gpn/tps40057"
+			(at 115.57 71.12 0)
+			(hide yes)
+			(show_name no)
+			(do_not_autoplace no)
+			(effects
+				(font
+					(size 1.27 1.27)
+					(italic yes)
+				)
+			)
+		)
+		(property "Description" ""
+			(at 115.57 71.12 0)
+			(hide yes)
+			(show_name no)
+			(do_not_autoplace no)
+			(effects
+				(font
+					(size 1.27 1.27)
+				)
+			)
+		)
+		(pin "4"
+		)
+		(pin "12"
+		)
+		(pin "13"
+		)
+		(pin "5"
+		)
+		(pin "9"
+		)
+		(pin "11"
+		)
+		(pin "14"
+		)
+		(pin "7"
+		)
+		(pin "EPAD"
+		)
+		(pin "3"
+		)
+		(pin "1"
+		)
+		(pin "6"
+		)
+		(pin "10"
+		)
+		(pin "15"
+		)
+		(pin "8"
+		)
+		(pin "2"
+		)
+		(pin "16"
+		)
+		(instances
+			(project "PDcharger"
+				(path "/e5ca95e5-7645-46ed-9827-1ed4c9d3ad41"
+					(reference "U1")
+					(unit 1)
+				)
+			)
+		)
+	)
 	(sheet_instances
 		(path "/"

Commit message: add
Parts:
- removed U1: TPS40057PWPR, TPS40057PWPR_footprints:PWP16_2P31X2P46-M, symbol 2026-06-10_10-14-18:TPS40057PWPR
- added C1, C3: 100nF, symbol Device:C
- added C2, C4: 1μF, symbol Device:C
- added C5, C6: 390pF, symbol Device:C
- added IC1: CYPD3175-24LQXQ, QFN50P400X400X60-25N-D, symbol CYPD3175-24LQXQ:CYPD3175-24LQXQ
- added J1: UJ20-C-H-G-SMT-1-P16-TR, UJ20-C-H-G-SMT-1-P16-TR:SAMESKY_UJ20-C-H-G-SMT-1-P16-TR, symbol UJ20-C-H-G-SMT-1-P16-TR:UJ20-C-H-G-SMT-1-P16-TR
- added R1: 5mΩ, symbol Device:R
- added R2: R, symbol Device:R
Connections:
- new net: C2.2, IC1.24 (VCCD)
- new net: IC1.20 (FB), R2.2
- new net: C3.2, C4.2, IC1.23 (VDDD)
- new net: C1.2, IC1.21 (CATH/COMP)
- new net CC1: C5.1, IC1.15 (CC1), J1.A5 (CC1)
- new net CC2: C6.1, IC1.14 (CC2), J1.B5 (CC2)
- new net CSP: IC1.19 (CSP), J1.A1_B12 (GND), J1.B1_A12 (GND__1), R1.1
- new net DN: IC1.16 (DM0/GPIO), J1.B7 (DN2)
- new net DP: IC1.17 (DP0/GPIO), J1.A6 (DP1), J1.B6 (DP2)
- new net GND: C1.1, C2.1, C3.1, C4.1, C5.2, C6.2, IC1.22 (GND), IC1.25 (EPAD), R1.2, R2.1
- new net VBUS: IC1.11 (VBUS_C_MON_DISCHARGE), J1.A4_B9 (VBUS), J1.B4_A9 (VBUS__1)

Commit message: add
Parts:
- added U1: TPS40057PWPR, PWP16_2P31X2P46, symbol 2026-06-10_10-14-18:TPS40057PWPR
Connections:
- new net 24VDC: U1.15 (VIN)
Changed lines of the file:
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@@
+		)
+	)
+	(label "24VDC"
+		(at 128.27 83.82 0)
+		(effects
+			(font
+				(size 1.27 1.27)
+			)
+			(justify left bottom)
 		)
 	)
@@
 					(unit 1)
 				)
+			)
+		)
+	)
+	(symbol
+		(lib_id "2026-06-10_10-14-18:TPS40057PWPR")
+		(at 62.23 78.74 0)
+		(unit 1)
+		(body_style 1)
+		(exclude_from_sim no)
+		(in_bom yes)
+		(on_board yes)
+		(in_pos_files yes)
+		(dnp no)
+		(fields_autoplaced yes)
+		(property "Reference" "U1"
+			(at 95.25 68.58 0)
+			(show_name no)
+			(do_not_autoplace no)
+			(effects
+				(font
+					(size 1.524 1.524)
+				)
+			)
+		)
+		(property "Value" "TPS40057PWPR"
+			(at 95.25 71.12 0)
+			(show_name no)
+			(do_not_autoplace no)
+			(effects
+				(font
+					(size 1.524 1.524)
+				)
+			)
+		)
+		(property "Footprint" "PWP16_2P31X2P46"
+			(at 62.23 78.74 0)
+			(hide yes)
+			(show_name no)
+			(do_not_autoplace no)
+			(effects
+				(font
+					(size 1.27 1.27)
+					(italic yes)
+				)
+			)
+		)
+		(property "Datasheet" "https://www.ti.com/lit/gpn/tps40057"
+			(at 62.23 78.74 0)
+			(hide yes)
+			(show_name no)
+			(do_not_autoplace no)
+			(effects
+				(font
+					(size 1.27 1.27)
+					(italic yes)
+				)
+			)
+		)
+		(property "Description" ""
+			(at 62.23 78.74 0)
+			(hide yes)
+			(show_name no)
+			(do_not_autoplace no)
+			(effects
+				(font
+					(size 1.27 1.27)
+				)
+			)
+		)
+		(pin "5"
+		)
+		(pin "4"
+		)
+		(pin "7"
+		)
+		(pin "3"
+		)
+		(pin "8"
+		)
+		(pin "14"
+		)
+		(pin "6"
+		)
+		(pin "11"
+		)
+		(pin "16"
+		)
+		(pin "10"
+		)
+		(pin "15"
+		)
+		(pin "1"
+		)
+		(pin "12"
+		)
+		(pin "9"
+		)
+		(pin "EPAD"
+		)
+		(pin "2"
+		)
+		(pin "13"
+		)
+		(instances
+			(project "PDcharger"
+				(path "/e5ca95e5-7645-46ed-9827-1ed4c9d3ad41"
+					(reference "U1")
+					(unit 1)
+				)
